File: board-schematic/night-lamp.brd (EAGLE design)
At the start: 20.3 x 41.6 mm, 18 parts, among them IC1 TINY13-20SSU, Q1 MMBF170, U1 1825096-1

Commit message: Update schematics
Add a resistor between GND and ADC3 (pin 2) on ATtiny. This change is
needed to create a voltage divider between +5V and GND, where the ADC
measures its output.
Parts:
- added R8: 1M, rcl:R1206
- C1: value (none) -> 100n
- R1, R2, R3, R4: value (none) -> 180R
- R5: value (none) -> 8M2
- R6, R7: value (none) -> 15k
- moved PH1 1.91 mm to (5.84, 10.8)
Connections:
- net N$12: now also R8.2
- net N$2: now also R8.1
Routing:
- net N$2: track 47.0 -> 50.7 mm
- net N$12: track 2.33 -> 4.72 mm
- net N$1: track 56.0 -> 57.5 mm
Other:
- board size 20.3 x 41.6 mm -> 21.6 x 41.6 mm
